Commit message: cleaned sick urdf

File: src/sweepy_bringup/urdf/sick.xacro (robot description, xacro)
@@ -3,21 +3,21 @@
     <xacro:property name="realsense_offset_z" value=".210"/>    <!--8.25" (center of realsense to chasis low point)-->
     <link name="sick_link">
-    <visual>
-        <origin xyz="${.057/2} 0 0" rpy="0 0 0"/>
-        <geometry>
-        <box size="0.057 0.057 0.089"/>
-        </geometry>
-    </visual>
-    <collision>
-        <origin xyz="0 0 0" rpy="0 0 0"/>
-        <geometry>
-        <box size="0.057 0.057 0.089"/>
-        </geometry>
-    </collision>
-    <inertial>
-        <origin xyz="0 0 0" rpy="0 0 0"/>
-        <mass value="0.035"/>
-        <inertia ixx="0.001"  ixy="0"  ixz="0" iyy="0.001" iyz="0" izz="0.001" />
-    </inertial>
+        <visual>
+            <origin xyz="${.057/2} 0 0" rpy="0 0 0"/>
+            <geometry>
+            <box size="0.057 0.057 0.089"/>
+            </geometry>
+        </visual>
+        <collision>
+            <origin xyz="0 0 0" rpy="0 0 0"/>
+            <geometry>
+            <box size="0.057 0.057 0.089"/>
+            </geometry>
+        </collision>
+        <inertial>
+            <origin xyz="0 0 0" rpy="0 0 0"/>
+            <mass value="0.035"/>
+            <inertia ixx="0.001"  ixy="0"  ixz="0" iyy="0.001" iyz="0" izz="0.001" />
+        </inertial>
     </link>
     <joint name="sick_joint" type="fixed">
@@ -26,9 +26,3 @@
         <origin xyz=".813 0 .127" rpy="0 0 0"/>
     </joint>
-    <link name="sick_lidar_frame"/>
-    <joint name="sick_frame_joint" type="fixed">
-        <origin xyz="0 0 0" rpy="0 0 0"/>
-        <parent link="sick_link"/>
-        <child link="sick_lidar_frame"/>
-    </joint>
 </robot>
