Commit message: added camera in URDF

File: src/sweepy_bringup/urdf/gazebo_robot.urdf.xacro (robot description, xacro)
@@ -4,4 +4,9 @@
   <xacro:include filename="$(find sweepy_bringup)/urdf/gazebo_control.xacro"/>
   <xacro:include filename="$(find sweepy_bringup)/urdf/sensor_sick.xacro"/>
+  <xacro:include filename="$(find sweepy_bringup)/urdf/sensor_d455.urdf.xacro"/>
   <xacro:include filename="$(find sweepy_bringup)/urdf/gazebo_sensors.xacro"/>
+  <!-- Mount the D455 on base_link -->
+  <xacro:sensor_d455 parent="base_link" name="d455" use_nominal_extrinsics="true">
+    <origin xyz="0.8 0 0.45" rpy="0 0 0"/>
+  </xacro:sensor_d455>
 </robot>

File: src/sweepy_bringup/urdf/sensor_d455.urdf.xacro (robot description, xacro)
@@ -21,6 +21,6 @@
 <robot name="sensor_d455" xmlns:xacro="http://ros.org/wiki/xacro">
   <!-- Includes -->
-  <xacro:include filename="$(find realsense2_description)/urdf/_materials.urdf.xacro" />
-  <xacro:include filename="$(find realsense2_description)/urdf/_usb_plug.urdf.xacro" />
+  <xacro:include filename="$(find sweepy_bringup)/urdf/sensor_d455_materials.urdf.xacro" />
+  <xacro:include filename="$(find sweepy_bringup)/urdf/sensor_d455_usb_plug.urdf.xacro" />
   <xacro:macro name="sensor_d455" params="parent *origin name:=camera use_nominal_extrinsics:=false">
     <xacro:arg name="add_plug" default="false" />
