Commit message: Gazebo & RViz color rendering and added LiDAR mesh

File: src/sweepy_bringup/urdf/robot_core.xacro (robot description, xacro)
@@ -19,10 +19,10 @@
   <!-- chasis bottom point is the back bottom metal frame near the motors -->
   <!-- mass inaccurate, only matters for simulation -->
-  <!-- colors -->
+  <!-- colors for RViz visualization-->
   <material name="white">
     <color rgba="1 1 1 1" />
   </material>
   <material name="orange">
-    <color rgba="1 .3 .1 1" />
+    <color rgba="1 .3 .1 0.7" />
   </material>
   <material name="blue">
@@ -30,5 +30,5 @@
   </material>
   <material name="black">
-    <color rgba="0 0 0 1" />
+    <color rgba="0 0 0 0.7" />
   </material>
   <material name="red">
@@ -83,5 +83,5 @@
               <cylinder radius="${wheel_radius}" length="${wheel_thickness}"/>
           </geometry>
-          <material name="blue"/>
+          <material name="black"/>
       </visual>
       <collision>
@@ -95,5 +95,5 @@
   </link>
   <gazebo reference="left_wheel">
-      <material>Gazebo/Blue</material>
+      <material>Gazebo/Black</material>
   </gazebo>
   <!-- RIGHT WHEEL LINK -->
@@ -109,5 +109,5 @@
               <cylinder radius="${wheel_radius}" length="${wheel_thickness}"/>
           </geometry>
-          <material name="blue"/>
+          <material name="black"/>
       </visual>
       <collision>
@@ -121,5 +121,5 @@
   </link>
   <gazebo reference="right_wheel">
-      <material>Gazebo/Blue</material>
+      <material>Gazebo/Black</material>
   </gazebo>
   <!-- CASTER WHEEL LINK -->

File: src/sweepy_bringup/urdf/sensor_d455.urdf.xacro (robot description, xacro)
@@ -85,4 +85,7 @@
       </inertial>
     </link>
+    <gazebo reference="${name}_link">
+        <material>Gazebo/Grey</material>
+    </gazebo>
     <!-- Use the nominal extrinsics between camera frames if the calibrated extrinsics aren't being published. e.g. running the device in simulation  -->
     <xacro:if value="${use_nominal_extrinsics}">

File: src/sweepy_bringup/urdf/sensor_sick.xacro (robot description, xacro)
@@ -1,16 +1,21 @@
 <?xml version="1.0"?>
 <robot name="sweeper" xmlns:xacro="http://ros.org/wiki/xacro">
-    <xacro:property name="realsense_offset_z" value=".210"/>    <!--8.25" (center of realsense to chasis low point)-->
+    <!-- <xacro:property name="realsense_offset_z" value=".210"/>    8.25" (center of realsense to chasis low point) -->
+    <material name="grey">
+        <color rgba="0.5 0.5 0.5 1" />
+    </material>
     <link name="sick_link">
         <visual>
-            <origin xyz="${.057/2} 0 0" rpy="0 0 0"/>
+            <origin xyz="0 0 0" rpy="0 0 0"/>
             <geometry>
-            <box size="0.057 0.057 0.089"/>
+                <!-- <box size="0.057 0.057 0.089"/> -->
+                <mesh filename="file://$(find sweepy_bringup)/meshes/sick781.stl" />
             </geometry>
+            <material name="grey"/>
         </visual>
         <collision>
-            <origin xyz="0 0 0" rpy="0 0 0"/>
+            <origin xyz="-0.00 0 -0.02" rpy="0 0 0"/>
             <geometry>
-            <box size="0.057 0.057 0.089"/>
+                <box size="0.057 0.057 0.089"/>
             </geometry>
         </collision>
@@ -24,5 +29,8 @@
         <parent link="base_link"/>
         <child link="sick_link"/>
-        <origin xyz=".813 0 .127" rpy="0 0 0"/>
+        <origin xyz=".858 0 .127" rpy="0 0 0"/>
     </joint>
+    <gazebo reference="sick_link">
+        <material>Gazebo/Grey</material>
+    </gazebo>
 </robot>

Commit message: rm unused coloring

File: src/sweepy_bringup/urdf/robot_core.xacro (robot description, xacro)
@@ -20,18 +20,9 @@
   <!-- mass inaccurate, only matters for simulation -->
   <!-- colors for RViz visualization-->
-  <material name="white">
-    <color rgba="1 1 1 1" />
-  </material>
   <material name="orange">
     <color rgba="1 .3 .1 0.7" />
   </material>
-  <material name="blue">
-    <color rgba=".2 .2 1 1" />
-  </material>
   <material name="black">
     <color rgba="0 0 0 0.7" />
-  </material>
-  <material name="red">
-    <color rgba="1 0 0 1" />
   </material>
   <!-- base link-->
@@ -134,5 +125,5 @@
               <sphere radius="${caster_wheel_radius}"/>
           </geometry>
-          <material name="white"/>
+          <material name="black"/>
       </visual>
       <collision>
@@ -146,5 +137,5 @@
   </link>
   <gazebo reference="caster_wheel">
-      <material>Gazebo/White</material>
+      <material>Gazebo/Black</material>
       <mu1 value="0.001"/>
       <mu2 value="0.001"/>
