Commit message: updated base_footprint frame

File: src/sucky_bringup/urdf/robot_core.xacro (robot description, xacro)
@@ -33,5 +33,5 @@
     <parent link="base_link"/>
     <child link="base_footprint"/>
-    <origin xyz="0 0 0" rpy="0 0 0"/>
+    <origin xyz="0 0 -0.127" rpy="0 0 0"/>
   </joint>
   <!-- chassis link -->
