Commit message: updated lidar placement

File: src/sucky_bringup/urdf/sensor_sick_sucky.xacro (robot description, xacro)
@@ -29,5 +29,5 @@
         <parent link="base_link"/>
         <child link="sick_link"/>
-        <origin xyz=".24 0 .10" rpy="${pi} 0 0"/>
+        <origin xyz=".25 0 .10" rpy="${pi} 0 0"/>
     </joint>
     <gazebo reference="sick_link">
