Commit message: sucky urdf adjustments

File: src/sucky_bringup/urdf/robot_core_sucky.xacro (robot description, xacro)
@@ -6,20 +6,17 @@
   <xacro:property name="chassis_length" value="0.69"/>
   <xacro:property name="chassis_height" value="1.26"/>
-  <xacro:property name="chassis_mass" value="5"/>
+  <xacro:property name="chassis_mass" value="15"/>
   <xacro:property name="wheel_radius" value="0.127"/>
   <xacro:property name="wheel_thickness" value="0.038862"/>
   <xacro:property name="wheel_offset_y" value=".287147"/>
-  <xacro:property name="wheel_offset_z" value="0.0"/> <!--not used-->
-  <xacro:property name="wheel_offset_x" value="0.0"/> <!--not used-->
+  <xacro:property name="wheel_offset_z" value="0.0"/>
+  <xacro:property name="wheel_offset_x" value="-0.03"/> <!--Try to minimize this value to compensate for tilting of robot-->
   <xacro:property name="wheel_mass" value=".5"/>
-  <!-- <xacro:property name="caster_wheel_mass" value=".2"/>
-  <xacro:property name="caster_wheel_radius" value="0.0762"/>
-  <xacro:property name="caster_wheel_offset_z" value="0.0445"/>
-  <xacro:property name="caster_wheel_offset_x" value=".597"/> -->
   <xacro:property name="omni_wheel_mass" value=".2"/>
   <xacro:property name="omni_wheel_radius" value="0.0635"/> <!-- 2.5"-->
   <xacro:property name="omni_wheel_thickness" value="0.04"/>
   <xacro:property name="omni_wheel_offset_z" value="0.0635"/> <!-- (2.5") center of wheel to center of main axle-->
-  <xacro:property name="omni_wheel_offset_x" value="0.2406396"/> <!-- (9.474") center of wheel to center of main axle-->
+  <!-- <xacro:property name="omni_wheel_offset_x" value="0.2406396"/> (9.474") center of wheel to center of main axle -->
+  <xacro:property name="omni_wheel_offset_x" value="0.3146396"/> <!-- (9.474") center of wheel to center of main axle-->
   <xacro:property name="omni_wheel_offset_y" value="0.2752344"/> <!-- (10.836") center of wheel to center of main axle -->
   <!-- chasis bottom point is the back bottom metal frame near the motors -->
@@ -74,9 +71,10 @@
       <parent link="base_link"/>
       <child link="left_wheel"/>
-      <origin xyz="0 ${wheel_offset_y} 0" rpy="0 0 0" />
+      <origin xyz="${wheel_offset_x} ${wheel_offset_y} 0" rpy="0 0 0" />
       <axis xyz="0 1 0"/>
   </joint>
   <link name="left_wheel">
       <visual>
+          <origin xyz="0 0 0" rpy="0 0 0"/>
           <geometry>
               <!-- <cylinder radius="${wheel_radius}" length="${wheel_thickness}"/> -->
@@ -103,5 +101,5 @@
       <parent link="base_link"/>
       <child link="right_wheel"/>
-      <origin xyz="0 ${-wheel_offset_y} 0" rpy="0 0 ${pi}" />
+      <origin xyz="${wheel_offset_x} ${-wheel_offset_y} 0" rpy="0 0 ${pi}" />
       <axis xyz="0 -1 0"/>
   </joint>
@@ -126,26 +124,4 @@
       <material>Gazebo/Black</material>
   </gazebo>
-  <!-- CASTER WHEEL LINK -->
-  <!-- <joint name="caster_wheel_joint" type="fixed">
-      <parent link="chassis"/>
-      <child link="caster_wheel"/>
-      <origin xyz="${caster_wheel_offset_x} 0 ${caster_wheel_offset_z}"/>
-  </joint>
-  <link name="caster_wheel">
-      <visual>
-          <geometry>
-              <sphere radius="${caster_wheel_radius}"/>
-          </geometry>
-          <material name="black"/>
-      </visual>
-      <collision>
-          <geometry>
-              <sphere radius="${caster_wheel_radius}"/>
-          </geometry>
-      </collision>
-      <xacro:inertial_sphere mass="${caster_wheel_mass}" radius="${caster_wheel_radius}">
-          <origin xyz="0 0 0" rpy="0 0 0"/>
-      </xacro:inertial_sphere>
-  </link> -->
   <!-- LEFT OMNI WHEEL LINK -->
   <joint name="left_omni_wheel_joint" type="fixed">

Commit message: increased sucky mass

File: src/sucky_bringup/urdf/robot_core_sucky.xacro (robot description, xacro)
@@ -6,5 +6,5 @@
   <xacro:property name="chassis_length" value="0.69"/>
   <xacro:property name="chassis_height" value="1.26"/>
-  <xacro:property name="chassis_mass" value="15"/>
+  <xacro:property name="chassis_mass" value="40"/>
   <xacro:property name="wheel_radius" value="0.127"/>
   <xacro:property name="wheel_thickness" value="0.038862"/>
